File: ns-1.kicad_pcb (KiCad board)
At the start: 4 copper layers, 172 x 135 mm, 74 parts, among them J1 AudioJack3, J2 AudioJack2, J3 AudioJack2, J4 AudioJack2, J5 AudioJack2, J6 Conn_01x11, J7 USB_C_Receptacle_USB2.0_16P, SW1 SW_Push_45deg, SW10 SW_Push_45deg, SW11 SW_Push_45deg, SW12 SW_Push_45deg, SW13 SW_Push_45deg, SW14 SW_Push_45deg, SW15 SW_Push_45deg, SW16 SW_Push_45deg, SW17 SW_Push_45deg, SW18 SW_Push_45deg, SW19 SW_Push_45deg, SW2 RotaryEncoder_Switch_MP, SW20 SW_Push, SW3 SW_Push_45deg, SW4 SW_Push_45deg, SW5 RotaryEncoder_Switch_MP, SW6 SW_Push_45deg, SW7 RotaryEncoder_Switch_MP, SW8 SW_Push_45deg, SW9 SW_Push_45deg, U1 Teensy4.1, U2 Teensy4.0_AudioShield_REVD

Commit message: update usb-c footprint
Parts:
- J7: footprint Connector_USB:USB_C_Receptacle_Amphenol_12401948E412A -> Connector_USB:USB_C_Receptacle_HRO_TYPE-C-31-M-12
- SW1, SW10, SW11, SW12, SW13, SW14, SW15, SW16, SW17, SW18, SW19, SW20, SW3, SW4, SW6, SW8, SW9: footprint Button_Switch_Keyboard:SW_Cherry_MX_1.00u_PCB -> switches:SW_Cherry_MX_1.00u_PCB
- moved J7 5.10 mm to (76.3, 92.7)
- moved FB1 5.10 mm to (76.4, 83.3)
- moved R1 5.10 mm to (84.4, 91.1)
- moved R2 5.10 mm to (84.7, 94.6)
Routing:
- net /D+: track 21.0 -> 28.3 mm
- net /D-: track 20.7 -> 26.4 mm
- net +5V: track 59.2 -> 56.6 mm
- net Net-(J7-SHIELD): track 23.9 -> 21.4 mm
- net GND: track 94.5 -> 96.8 mm
- net Net-(J7-CC2): track 2.45 -> 3.50 mm
- net Net-(J7-CC1): track 2.37 -> 3.43 mm
