File: ns-1.kicad_sch (KiCad schematic)
At the start: 66 parts, among them J6 Conn_01x11, J7 USB_C_Receptacle_USB2.0_16P, SW1 SW_Push_45deg, SW10 SW_Push_45deg, SW11 SW_Push_45deg, SW12 SW_Push_45deg, SW13 SW_Push_45deg, SW14 SW_Push_45deg, SW15 SW_Push_45deg, SW16 SW_Push_45deg, SW17 SW_Push_45deg, SW18 SW_Push_45deg, SW19 SW_Push_45deg, SW2 RotaryEncoder_Switch_MP, SW20 SW_Push, SW3 SW_Push_45deg, SW4 SW_Push_45deg, SW5 RotaryEncoder_Switch_MP, SW6 SW_Push_45deg, SW7 RotaryEncoder_Switch_MP, SW8 SW_Push_45deg, SW9 SW_Push_45deg, U1 Teensy4.1

Commit message: update usb-c footprint
Parts:
- C2, C3, C4, C6: LCSC PN (none) -> C22435941
- D1, D10, D11, D12, D13, D14, D15, D16, D2, D3, D4, D5, D6, D7, D8, D9: LCSC PN (none) -> C917030
- FB1: LCSC PN (none) -> C2943443
- J7: footprint Connector_USB:USB_C_Receptacle_Amphenol_12401948E412A -> Connector_USB:USB_C_Receptacle_HRO_TYPE-C-31-M-12; LCSC PN (none) -> C3197899
- R1, R2: LCSC PN (none) -> C2906874
- R3: LCSC PN (none) -> C317926
- R4, R5, R6, R7, R8: LCSC PN (none) -> C122970
