File: hardware/ns-1.kicad_pcb (KiCad board)
At the start: 4 copper layers, 172 x 145.6 mm, 142 parts, among them J1 Micro_SD_Card_Det2, J10 AudioJack2, J11 AudioJack2, J12 AudioJack2, J13 AudioJack2, J6 Conn_01x11, J7 USB_C_Receptacle_USB2.0_16P, J8 Conn_ARM_JTAG_SWD_10, J9 AudioJack3, SW1 SW_Push_45deg, SW10 SW_Push_45deg, SW11 SW_Push_45deg, SW12 SW_Push_45deg, SW13 SW_Push_45deg, SW14 SW_Push_45deg, SW15 SW_Push_45deg, SW16 SW_Push_45deg, SW17 SW_Push_45deg, SW18 SW_Push_45deg, SW19 SW_Push_45deg, SW2 RotaryEncoder_Switch_MP, SW20 SW_Push, SW21 SW_Push, SW22 SW_Push, SW3 SW_Push_45deg, SW4 SW_Push_45deg, SW5 RotaryEncoder_Switch_MP, SW6 SW_Push_45deg, SW7 RotaryEncoder_Switch_MP, SW8 SW_Push_45deg, SW9 SW_Push_45deg, U1 APS6404L-3SQRx-SN, U2 XC6206P182MR, U3 STM32H723ZGTx, U4 SGTL5000XNLA3, U5 USBLC6-2P6, U6 AP7361C-33E, U7 APS6404L-3SQRx-SN, Y1 25MHz

Commit message: finish layout
Parts:
- added C49: 100n, Capacitor_SMD:C_0402_1005Metric, F.Cu at (176.7, 26.1)
- added C50: 1u, Capacitor_SMD:C_0402_1005Metric, F.Cu at (174.1, 26.1)
- added G***: LOGO, LOGO, F.Cu at (94.8, 58.4)
- added G***: LOGO, LOGO, F.Cu at (95.7, 155.0)
- added U8: ER_OLEDM0.91_1x-I2C, Display:ER_OLEDM0.91_1x-I2C, F.Cu at (172.5, 28.6)
- moved G*** 6.57 mm to (190.7, 74.4)
- moved C3 0.99 mm to (207.1, 33.8), turned to 45 degrees
- moved R8 0.80 mm to (222.0, 122.5)
- moved C12 0.50 mm to (200.2, 57.4)
- moved C14 0.19 mm to (208.3, 35.2)
Connections:
- net /SGTL5000/SCL renamed /SCL
- net /SGTL5000/SDA renamed /SDA
- U3 pad 114: /Peripherals/S1 -> unconnected-(U3-PD0-Pad114)
- U3 pad 115: /Peripherals/S2 -> unconnected-(U3-PD1-Pad115)
- U3 pad 118: /Peripherals/COL0 -> /Peripherals/COL3
- U3 pad 119: /Peripherals/COL1 -> /Peripherals/COL2
- U3 pad 122: /Peripherals/COL2 -> /Peripherals/COL1
- U3 pad 123: /Peripherals/COL3 -> /Peripherals/COL0
- U3 pad 64: /Peripherals/B1 -> unconnected-(U3-PE11-Pad64)
- U3 pad 65: /Peripherals/A1 -> unconnected-(U3-PE12-Pad65)
- U3 pad 88: unconnected-(U3-PG3-Pad88) -> /Peripherals/A2
- U3 pad 89: unconnected-(U3-PG4-Pad89) -> /Peripherals/B2
- U3 pad 90: unconnected-(U3-PG5-Pad90) -> /Peripherals/S2
- U3 pad 91: unconnected-(U3-PG6-Pad91) -> /Peripherals/B1
- U3 pad 92: unconnected-(U3-PG7-Pad92) -> /Peripherals/A1
- U3 pad 93: unconnected-(U3-PG8-Pad93) -> /Peripherals/S1
- U3 pad 96: /Peripherals/A2 -> unconnected-(U3-PC6-Pad96)
- U3 pad 97: /Peripherals/B2 -> unconnected-(U3-PC7-Pad97)
Routing:
- net /Peripherals/COL0: track 0.00 -> 186.2 mm, vias 0 -> 1
- net /Peripherals/ROW3: track 0.00 -> 173.0 mm, vias 0 -> 1
- net /Peripherals/COL1: track 0.00 -> 166.6 mm, vias 0 -> 1
- net /Peripherals/BTN1: track 0.00 -> 157.5 mm, vias 0 -> 2
- net /Peripherals/ROW2: track 0.00 -> 154.1 mm, vias 0 -> 1
- net /Peripherals/COL2: track 0.00 -> 153.0 mm, vias 0 -> 1
- net /Peripherals/VSK: track 1.38 -> 152.4 mm, vias 0 -> 2
- net /Power/D-: track 2.27 -> 141.4 mm, vias 1 -> 2
- net /Power/D+: track 2.27 -> 138.3 mm, vias 1 -> 2
- net /Peripherals/ROW1: track 0.00 -> 135.2 mm, vias 0 -> 1
- net /Peripherals/COL3: track 0.00 -> 131.3 mm, vias 0 -> 1
- net /Peripherals/POT1: track 8.82 -> 139.1 mm, vias 2 -> 3
- net /Peripherals/POT2: track 5.16 -> 127.6 mm, vias 0 -> 2
- net /Peripherals/B3: track 0.00 -> 116.4 mm
- net /Peripherals/ROW0: track 0.00 -> 116.3 mm, vias 0 -> 1
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Other:
- board text added: "ATTIRE AJUAF BLEUES FRRT IRO ROB"
- board text removed: "RST"

Commit message: finalize respin
Parts:
- J9: footprint Connector_Audio:Jack_3.5mm_CUI_SJ1-3533NG_Horizontal -> Connector_Audio:Jack_3.5mm_CUI_SJ-3523-SMT_Horizontal
- moved J9 3.80 mm to (79.8, 150.6)
Routing:
- net Net-(U4-HP_L): track 113.4 -> 124.0 mm
- net Net-(U4-HP_R): track 113.9 -> 109.5 mm, vias 1 -> 2
- net Net-(U4-HP_VGND): track 113.3 -> 117.0 mm, vias 1 -> 2
