File: hardware/peripherals.kicad_sch (KiCad schematic)
At the start: 53 parts, among them J6 Conn_01x11, SW1 SW_Push_45deg, SW10 SW_Push_45deg, SW11 SW_Push_45deg, SW12 SW_Push_45deg, SW13 SW_Push_45deg, SW14 SW_Push_45deg, SW15 SW_Push_45deg, SW16 SW_Push_45deg, SW17 SW_Push_45deg, SW18 SW_Push_45deg, SW19 SW_Push_45deg, SW2 RotaryEncoder_Switch_MP, SW20 SW_Push, SW3 SW_Push_45deg, SW4 SW_Push_45deg, SW5 RotaryEncoder_Switch_MP, SW6 SW_Push_45deg, SW7 RotaryEncoder_Switch_MP, SW8 SW_Push_45deg, SW9 SW_Push_45deg

Commit message: start rearranging layout
Parts:
- RV5: footprint Potentiometer_THT:Potentiometer_Bourns_PTA4543_Single_Slide -> Potentiometer_THT:Potentiometer_Alps_RK09K_Single_Vertical
Connections:
- net SL1 renamed VSK
Changed lines of the file:
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@@
 	(wire
 		(pts
-			(xy 242.57 109.22) (xy 242.57 119.38)
+			(xy 237.49 109.22) (xy 237.49 119.38)
 		)
 		(stroke
@@
 	(wire
 		(pts
-			(xy 203.2 109.22) (xy 203.2 119.38)
+			(xy 198.12 109.22) (xy 198.12 119.38)
 		)
 		(stroke
@@
 	(wire
 		(pts
-			(xy 208.28 109.22) (xy 203.2 109.22)
+			(xy 208.28 109.22) (xy 198.12 109.22)
 		)
 		(stroke
@@
 	(wire
 		(pts
-			(xy 167.64 109.22) (xy 162.56 109.22)
+			(xy 167.64 109.22) (xy 157.48 109.22)
 		)
 		(stroke
@@
 	(wire
 		(pts
-			(xy 242.57 119.38) (xy 255.27 119.38)
+			(xy 237.49 119.38) (xy 255.27 119.38)
 		)
 		(stroke
@@
 	(wire
 		(pts
-			(xy 162.56 109.22) (xy 162.56 119.38)
+			(xy 157.48 109.22) (xy 157.48 119.38)
 		)
 		(stroke
@@
 	(wire
 		(pts
-			(xy 247.65 109.22) (xy 242.57 109.22)
+			(xy 247.65 109.22) (xy 237.49 109.22)
 		)
 		(stroke
@@
 	(wire
 		(pts
-			(xy 203.2 119.38) (xy 215.9 119.38)
+			(xy 198.12 119.38) (xy 215.9 119.38)
 		)
 		(stroke
@@
 	(wire
 		(pts
-			(xy 162.56 119.38) (xy 175.26 119.38)
+			(xy 157.48 119.38) (xy 175.26 119.38)
 		)
 		(stroke
@@
 		)
 	)
-	(label "A3"
-		(at 243.84 106.68 0)
+	(hierarchical_label "ROW1"
+		(shape bidirectional)
+		(at 121.92 83.82 0)
 		(effects
 			(font
 				(size 1.27 1.27)
 			)
-			(justify left bottom)
+			(justify left)
 		)
 	)
-	(label "S1"
-		(at 186.69 106.68 180)
+	(hierarchical_label "MISO"
+		(shape output)
+		(at 96.52 167.64 180)
 		(effects
 			(font
 				(size 1.27 1.27)
 			)
-			(justify right bottom)
+			(justify right)
 		)
 	)
-	(label "B1"
-		(at 163.83 111.76 0)
+	(hierarchical_label "A1"
+		(shape output)
+		(at 163.83 106.68 180)
 		(effects
 			(font
 				(size 1.27 1.27)
 			)
-			(justify left bottom)
+			(justify right)
 		)
 	)
-	(label "B2"
-		(at 204.47 111.76 0)
+	(hierarchical_label "POT2"
+		(shape output)
+		(at 198.12 43.18 90)
 		(effects
 			(font
 				(size 1.27 1.27)
 			)
-			(justify left bottom)
+			(justify left)
 		)
 	)
-	(label "POT3"
-		(at 223.52 43.18 180)
+	(hierarchical_label "B2"
+		(shape output)
+		(at 204.47 111.76 180)
 		(effects
 			(font
 				(size 1.27 1.27)
 			)
-			(justify right bottom)
+			(justify right)
 		)
 	)
-	(label "POT4"
-		(at 248.92 43.18 180)
+	(hierarchical_label "A3"
+		(shape output)
+		(at 243.84 106.68 180)
 		(effects
 			(font
 				(size 1.27 1.27)
 			)
-			(justify right bottom)
+			(justify right)
 		)
 	)
-	(label "POT2"
-		(at 198.12 43.18 180)
+	(hierarchical_label "POT4"
+		(shape output)
+		(at 248.92 43.18 90)
 		(effects
 			(font
 				(size 1.27 1.27)
 			)
-			(justify right bottom)
+			(justify left)
 		)
 	)
-	(label "B3"
-		(at 243.84 111.76 0)
+	(hierarchical_label "S2"
+		(shape output)
+		(at 227.33 106.68 0)
 		(effects
 			(font
 				(size 1.27 1.27)
 			)
-			(justify left bottom)
+			(justify left)
 		)
 	)
-	(label "POT1"
-		(at 172.72 43.18 180)
+	(hierarchical_label "POT3"
+		(shape output)
+		(at 223.52 43.18 90)
 		(effects
 			(font
 				(size 1.27 1.27)
 			)
-			(justify right bottom)
+			(justify left)
 		)
 	)
-	(label "S2"
-		(at 227.33 106.68 180)
+	(hierarchical_label "S1"
+		(shape output)
+		(at 186.69 106.68 0)
 		(effects
 			(font
 				(size 1.27 1.27)
 			)
-			(justify right bottom)
+			(justify left)
 		)
 	)
-	(label "A2"
-		(at 204.47 106.68 0)
+	(hierarchical_label "COL3"
+		(shape bidirectional)
+		(at 102.87 44.45 90)
 		(effects
 			(font
 				(size 1.27 1.27)
 			)
-			(justify left bottom)
+			(justify left)
 		)
 	)
-	(label "S3"
-		(at 266.7 106.68 180)
+	(hierarchical_label "DC"
+		(shape input)
+		(at 96.52 177.8 180)
 		(effects
 			(font
 				(size 1.27 1.27)
 			)
-			(justify right bottom)
+			(justify right)
 		)
 	)
-	(label "A1"
-		(at 163.83 106.68 0)
+	(hierarchical_label "S3"
+		(shape output)
+		(at 266.7 106.68 0)
 		(effects
 			(font
 				(size 1.27 1.27)
 			)
-			(justify left bottom)
+			(justify left)
 		)
 	)
-	(label "SL1"
-		(at 172.72 58.42 180)
+	(hierarchical_label "COL1"
+		(shape bidirectional)
+		(at 64.77 44.45 90)
 		(effects
 			(font
 				(size 1.27 1.27)
 			)
-			(justify right bottom)
+			(justify left)
 		)
 	)
-	(hierarchical_label "ROW1"
-		(shape bidirectional)
-		(at 121.92 83.82 0)
+	(hierarchical_label "RST"
+		(shape input)
+		(at 96.52 175.26 180)
 		(effects
 			(font
 				(size 1.27 1.27)
 			)
-			(justify left)
+			(justify right)
 		)
 	)
-	(hierarchical_label "MISO"
-		(shape output)
-		(at 96.52 167.64 180)
+	(hierarchical_label "ROW0"
+		(shape bidirectional)
+		(at 121.92 64.77 0)
 		(effects
 			(font
 				(size 1.27 1.27)
 			)
-			(justify right)
+			(justify left)
 		)
 	)
-	(hierarchical_label "COL3"
+	(hierarchical_label "COL2"
 		(shape bidirectional)
-		(at 102.87 44.45 90)
+		(at 83.82 44.45 90)
 		(effects
 			(font
@@
 		)
 	)
-	(hierarchical_label "DC"
+	(hierarchical_label "MOSI"
 		(shape input)
-		(at 96.52 177.8 180)
+		(at 96.52 170.18 180)
 		(effects
 			(font
@@
 		)
 	)
-	(hierarchical_label "COL1"
+	(hierarchical_label "ROW2"
 		(shape bidirectional)
-		(at 64.77 44.45 90)
+		(at 121.92 102.87 0)
 		(effects
 			(font
@@
 		)
 	)
-	(hierarchical_label "RST"
+	(hierarchical_label "TCS"
 		(shape input)
-		(at 96.52 175.26 180)
+		(at 96.52 172.72 180)
 		(effects
 			(font
@@
 		)
 	)
-	(hierarchical_label "ROW0"
-		(shape bidirectional)
-		(at 121.92 64.77 0)
+	(hierarchical_label "A2"
+		(shape output)
+		(at 204.47 106.68 180)
 		(effects
 			(font
 				(size 1.27 1.27)
 			)
-			(justify left)
+			(justify right)
 		)
 	)
-	(hierarchical_label "COL2"
-		(shape bidirectional)
-		(at 83.82 44.45 90)
+	(hierarchical_label "B1"
+		(shape output)
+		(at 163.83 111.76 180)
 		(effects
 			(font
 				(size 1.27 1.27)
 			)
-			(justify left)
+			(justify right)
 		)
 	)
-	(hierarchical_label "MOSI"
-		(shape input)
-		(at 96.52 170.18 180)
+	(hierarchical_label "POT1"
+		(shape output)
+		(at 172.72 43.18 90)
 		(effects
 			(font
 				(size 1.27 1.27)
 			)
-			(justify right)
+			(justify left)
 		)
 	)
-	(hierarchical_label "ROW2"
+	(hierarchical_label "COL0"
 		(shape bidirectional)
-		(at 121.92 102.87 0)
+		(at 45.72 44.45 90)
 		(effects
 			(font
@@
 		)
 	)
-	(hierarchical_label "TCS"
-		(shape input)
-		(at 96.52 172.72 180)
+	(hierarchical_label "B3"
+		(shape output)
+		(at 243.84 111.76 180)
 		(effects
 			(font
@@
 		)
 	)
-	(hierarchical_label "COL0"
-		(shape bidirectional)
-		(at 45.72 44.45 90)
+	(hierarchical_label "VSK"
+		(shape output)
+		(at 172.72 58.42 0)
 		(effects
 			(font
@@
 			)
 		)
-		(property "Footprint" "Potentiometer_THT:Potentiometer_Bourns_PTA4543_Single_Slide"
+		(property "Footprint" "Potentiometer_THT:Potentiometer_Alps_RK09K_Single_Vertical"
 			(at 172.72 66.04 0)
 			(hide yes)

Commit message: finish placement, add sd, codec routing
Other:
- moved on the sheet: J6, R3, SW20

Commit message: finish layout
Parts:
- added C49: 100n, Capacitor_SMD:C_0402_1005Metric, symbol Device:C_Small_US
- added C50: 1u, Capacitor_SMD:C_0402_1005Metric, symbol Device:C_Small_US
- added U8: ER_OLEDM0.91_1x-I2C, Display:ER_OLEDM0.91_1x-I2C, symbol Display_Graphic:ER_OLEDM0.91_1x-I2C
Connections:
- net +3.3V: now also C49.1, C50.1, U8.2 (VCC)
- net GND: now also C49.2, C50.2, U8.1 (GND)
- new net SCL: U8.3 (SCL)
- new net SDA: U8.4 (SDA)
Other:
- note added: "SSD1306"
- moved on the sheet: J6, R3, SW20

Commit message: finalize respin
Parts:
- C49, C8: LCSC PN (none) -> C1525
- C50: LCSC PN (none) -> C52923
- J6, RV1, RV2, RV3, RV4, RV5, SW1, SW10, SW11, SW12, SW13, SW14, SW15, SW16, SW17, SW18, SW19, SW2, SW20, SW3, SW4, SW5, SW6, SW7, SW8, SW9, U8: now left out of the parts list
- R3: LCSC PN C317926 -> C25804
Changed lines of the file:
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@@
 			)
 		)
+		(property "LCSC PN" "C1525"
+			(at 144.78 158.75 0)
+			(hide yes)
+			(show_name no)
+			(do_not_autoplace no)
+			(effects
+				(font
+					(size 1.27 1.27)
+				)
+			)
+		)
 		(pin "2"
 		)
@@
 			)
 		)
+		(property "LCSC PN" "C52923"
+			(at 154.94 158.75 0)
+			(hide yes)
+			(show_name no)
+			(do_not_autoplace no)
+			(effects
+				(font
+					(size 1.27 1.27)
+				)
+			)
+		)
 		(pin "2"
 		)
@@
 		(body_style 1)
 		(exclude_from_sim no)
-		(in_bom yes)
+		(in_bom no)
 		(on_board yes)
 		(in_pos_files yes)
@@
 		(body_style 1)
 		(exclude_from_sim no)
-		(in_bom yes)
+		(in_bom no)
 		(on_board yes)
 		(in_pos_files yes)
@@
 		(body_style 1)
 		(exclude_from_sim no)
-		(in_bom yes)
+		(in_bom no)
 		(on_board yes)
 		(in_pos_files yes)
@@
 		(body_style 1)
 		(exclude_from_sim no)
-		(in_bom yes)
+		(in_bom no)
 		(on_board yes)
 		(in_pos_files yes)
@@
 		(body_style 1)
 		(exclude_from_sim no)
-		(in_bom yes)
+		(in_bom no)
 		(on_board yes)
 		(in_pos_files yes)
@@
 		(body_style 1)
 		(exclude_from_sim no)
-		(in_bom yes)
+		(in_bom no)
 		(on_board yes)
 		(in_pos_files yes)
@@
 		(body_style 1)
 		(exclude_from_sim no)
-		(in_bom yes)
+		(in_bom no)
 		(on_board yes)
 		(in_pos_files yes)
@@
 		(body_style 1)
 		(exclude_from_sim no)
-		(in_bom yes)
+		(in_bom no)
 		(on_board yes)
 		(in_pos_files yes)
@@
 			)
 		)
-		(property "LCSC PN" ""
+		(property "LCSC PN" "C1525"
 			(at 240.03 46.99 0)
 			(hide yes)
@@
 		(body_style 1)
 		(exclude_from_sim no)
-		(in_bom yes)
+		(in_bom no)
 		(on_board yes)
 		(in_pos_files yes)
@@
 		(body_style 1)
 		(exclude_from_sim no)
-		(in_bom yes)
+		(in_bom no)
 		(on_board yes)
 		(in_pos_files yes)
@@
 		(body_style 1)
 		(exclude_from_sim no)
-		(in_bom yes)
+		(in_bom no)
 		(on_board yes)
 		(in_pos_files yes)
@@
 		(body_style 1)
 		(exclude_from_sim no)
-		(in_bom yes)
+		(in_bom no)
 		(on_board yes)
 		(in_pos_files yes)
@@
 		(body_style 1)
 		(exclude_from_sim no)
-		(in_bom yes)
+		(in_bom no)
 		(on_board yes)
 		(in_pos_files yes)
@@
 		(body_style 1)
 		(exclude_from_sim no)
-		(in_bom yes)
+		(in_bom no)
 		(on_board yes)
 		(in_pos_files yes)
@@
 			)
 		)
-		(property "LCSC PN" "C317926"
+		(property "LCSC PN" "C25804"
 			(at 55.88 160.02 0)
 			(hide yes)
@@
 		(body_style 1)
 		(exclude_from_sim no)
-		(in_bom yes)
+		(in_bom no)
 		(on_board yes)
 		(in_pos_files yes)
@@
 		(body_style 1)
 		(exclude_from_sim no)
-		(in_bom yes)
+		(in_bom no)
 		(on_board yes)
 		(in_pos_files yes)
@@
 		(body_style 1)
 		(exclude_from_sim no)
-		(in_bom yes)
+		(in_bom no)
 		(on_board yes)
 		(in_pos_files yes)
@@
 		(body_style 1)
 		(exclude_from_sim no)
-		(in_bom yes)
+		(in_bom no)
 		(on_board yes)
 		(in_pos_files yes)
@@
 		(body_style 1)
 		(exclude_from_sim no)
-		(in_bom yes)
+		(in_bom no)
 		(on_board yes)
 		(in_pos_files yes)
@@
 		(body_style 1)
 		(exclude_from_sim no)
-		(in_bom yes)
+		(in_bom no)
 		(on_board yes)
 		(in_pos_files yes)
@@
 		(body_style 1)
 		(exclude_from_sim no)
-		(in_bom yes)
+		(in_bom no)
 		(on_board yes)
 		(in_pos_files yes)
@@
 		(body_style 1)
 		(exclude_from_sim no)
-		(in_bom yes)
+		(in_bom no)
 		(on_board yes)
 		(in_pos_files yes)
@@
 		(body_style 1)
 		(exclude_from_sim no)
-		(in_bom yes)
+		(in_bom no)
 		(on_board yes)
 		(in_pos_files yes)
@@
 		(body_style 1)
 		(exclude_from_sim no)
-		(in_bom yes)
+		(in_bom no)
 		(on_board yes)
 		(in_pos_files yes)
@@
 		(body_style 1)
 		(exclude_from_sim no)
-		(in_bom yes)
+		(in_bom no)
 		(on_board yes)
 		(in_pos_files yes)
@@
 		(body_style 1)
 		(exclude_from_sim no)
-		(in_bom yes)
+		(in_bom no)
 		(on_board yes)
 		(in_pos_files yes)
@@
 		(body_style 1)
 		(exclude_from_sim no)
-		(in_bom yes)
+		(in_bom no)
 		(on_board yes)
 		(in_pos_files yes)
